Commit message: fixed urdf for podi

File: tbd_podi_description/urdf/pioneer3dx.urdf.xacro (robot description, xacro)
@@ -5,10 +5,5 @@
     <!-- Chassis -->
     <link name="base_link">
-        <inertial>
-            <mass value="3.5"/>
-            <!--<origin xyz="-0.025 0 -0.223"/>-->
-            <origin xyz="0 0 0"/>
-            <inertia ixx="1" ixy="0" ixz="0" iyy="1" iyz="0" izz="1"/>
-        </inertial>
+        <xacro:box_inertial x="0.35" y="0.25" z="0.14" mass="10" />
         <visual>
             <origin xyz="-0.045 0 0.148" rpy="0 0 0"/>
@@ -210,20 +205,3 @@
         <top_plate parent="base_link"/>
     </create>
-    <gazebo>
-        <plugin name="differential_drive_controller" filename="libgazebo_ros_diff_drive.so">
-            <alwaysOn>true</alwaysOn>
-            <updateRate>100</updateRate>
-            <leftJoint>left_wheel_joint</leftJoint>
-            <rightJoint>right_wheel_joint</rightJoint>
-            <wheelSeparation>0.158</wheelSeparation>
-            <wheelDiameter>0.12</wheelDiameter>
-            <torque>5</torque>
-            <commandTopic>cmd_vel</commandTopic>
-            <robotBaseFrame>base_link</robotBaseFrame>
-            <odometryTopic>odom</odometryTopic>
-            <odometryFrame>odom</odometryFrame>
-        </plugin>
-        <!-- TODO include P3D (ground truth) plugin -->
-        <!-- XXX old urdf included a gazebo_ros_controller_manager plugin with a 1 second update rate -->
-    </gazebo>
 </robot>

File: tbd_podi_description/urdf/pioneer3dx_wheel.xacro (robot description, xacro)
@@ -56,7 +56,4 @@
     <joint name="${suffix}_wheel_joint" type="continuous">
       <axis xyz="0 1 0"/>
-      <anchor xyz="0 0 0"/>
-      <limit effort="100" velocity="100" />
-      <joint_properties damping="0.0" friction="0.0" />
       <origin xyz="0 ${reflect*0.158} 0.091" rpy="0 0 0"/>
       <parent link="${parent}"/>
@@ -64,4 +61,6 @@
     </joint>
     <!-- Transmission variable for gazebo -->
+    <!-- This is commented out because it is used by gazebo_ros_controller, it will superseed
+    the internal wheel controller if set
     <transmission type="pr2_mechanism_model/SimpleTransmission" name="${suffix}_wheel_trans">
       <type>transmission_interface/SimpleTransmission</type>
@@ -73,5 +72,5 @@
         <hardwareInterface>hardware_interface/VelocityJointInterface</hardwareInterface>
       </joint>
-    </transmission>
+    </transmission> -->
     <gazebo reference="${suffix}_hubcap">
       <material value="Gazebo/Yellow"/>

File: tbd_podi_description/urdf/podi.gazebo.xacro (robot description, xacro)
@@ -1,36 +1,66 @@
 <?xml version="1.0"?>
 <robot xmlns:xacro="http://ros.org/wiki/xacro">
-<gazebo reference="laser_scanner">
+  <gazebo>
+    <plugin name="differential_drive_controller" filename="libgazebo_ros_diff_drive.so">
+      <alwaysOn>true</alwaysOn>
+      <updateRate>100</updateRate>
+      <leftJoint>left_wheel_joint</leftJoint>
+      <rightJoint>right_wheel_joint</rightJoint>
+      <wheelSeparation>0.39</wheelSeparation>
+      <wheelDiameter>0.15</wheelDiameter>
+      <wheelTorque>20</wheelTorque>
+      <publishWheelJointState>true</publishWheelJointState>
+      <publishWheelTF>false</publishWheelTF>
+      <wheelAcceleration>1.8</wheelAcceleration>
+      <commandTopic>cmd_vel</commandTopic>
+      <robotBaseFrame>base_link</robotBaseFrame>
+      <odometryTopic>odom</odometryTopic>
+      <odometryFrame>odom</odometryFrame>
+      <odometrySource>encoder</odometrySource>      <!-- The options are world and encoder. World means getting it straight from Gazebo -->
+    </plugin>
+    <!-- ground truth -->
+    <plugin name="p3d_base_controller" filename="libgazebo_ros_p3d.so">
+      <alwaysOn>true</alwaysOn>
+      <updateRate>100.0</updateRate>
+      <bodyName>base_link</bodyName>
+      <topicName>pose_ground_truth</topicName>
+      <gaussianNoise>0.01</gaussianNoise>
+      <frameName>map</frameName>
+      <xyzOffsets>0 0 0</xyzOffsets>
+      <rpyOffsets>0 0 0</rpyOffsets>
+    </plugin>
+  </gazebo>
+  <gazebo reference="laser_scanner">
     <sensor type="gpu_ray" name="lms100x">
-        <pose>0 0 0 0 0 0</pose>
-        <!-- <visualize>false</visualize> -->
-        <update_rate>20</update_rate>
-        <ray>
-            <scan>
-                <horizontal>
-                    <samples>360</samples>
-                    <resolution>1</resolution>
-                    <min_angle>-1.570796</min_angle>
-                    <max_angle>1.570796</max_angle>
-                </horizontal>
-            </scan>
-            <range>
-                <min>0.10</min>
-                <max>30.0</max>
-                <resolution>0.01</resolution>
-            </range>
-            <noise>
-                <type>gaussian</type>
-                <mean>0.0</mean>
-                <stddev>0.01</stddev>
-            </noise>
-        </ray>
-        <plugin name="gazebo_ros_head_hokuyo_controller" filename="libgazebo_ros_gpu_laser.so">
-            <topicName>/scan</topicName>
-            <frameName>laser_scanner</frameName>
-        </plugin>
+      <pose>0 0 0 0 0 0</pose>
+      <!-- <visualize>false</visualize> -->
+      <update_rate>20</update_rate>
+      <ray>
+        <scan>
+          <horizontal>
+            <samples>360</samples>
+            <resolution>1</resolution>
+            <min_angle>-1.570796</min_angle>
+            <max_angle>1.570796</max_angle>
+          </horizontal>
+        </scan>
+        <range>
+          <min>0.10</min>
+          <max>30.0</max>
+          <resolution>0.01</resolution>
+        </range>
+        <noise>
+          <type>gaussian</type>
+          <mean>0.0</mean>
+          <stddev>0.01</stddev>
+        </noise>
+      </ray>
+      <plugin name="gazebo_ros_head_hokuyo_controller" filename="libgazebo_ros_gpu_laser.so">
+        <topicName>/scan</topicName>
+        <frameName>laser_scanner</frameName>
+      </plugin>
     </sensor>
-</gazebo>
-<gazebo reference="podi_display">
+  </gazebo>
+  <gazebo reference="podi_display">
     <visual>
       <plugin name="screen_video_controller" filename="libgazebo_ros_video.so">
@@ -40,5 +70,5 @@
       </plugin>
     </visual>
-</gazebo>
+  </gazebo>
   <gazebo reference="podi_front_camera">
     <sensor type="camera" name="front_camera">

File: tbd_podi_description/urdf/podi.urdf.xacro (robot description, xacro)
@@ -2,4 +2,6 @@
 <robot name="podi"
     xmlns:xacro="http://ros.org/wiki/xacro">
+    <!-- Inport inertia functions -->
+    <xacro:include filename="$(find tbd_podi_description)/urdf/inertia_tensors.xacro"/>
     <!-- Import the base robot -->
     <xacro:include filename="$(find tbd_podi_description)/urdf/pioneer3dx.urdf.xacro"/>

File: tbd_podi_description/urdf/podi_handle.xacro (robot description, xacro)
@@ -121,5 +121,5 @@
         <parent link="handle_base"/>
         <child link="handle_bottom_plate"/>
-        <limit lower="-1.57" upper="1.57" effort="0" velocity="1" />
+        <limit lower="-1.57" upper="1.57" effort="1" velocity="1" />
     </joint>
     <joint name="handle_bottom_plate_to_back_plate" type="fixed">

File: tbd_podi_description/urdf/podi_structure.xacro (robot description, xacro)
@@ -1,7 +1,4 @@
 <?xml version="1.0"?>
 <robot xmlns:xacro="http://ros.org/wiki/xacro">
-    <xacro:property name="laser_scanner_width" value="0.1" />
-    <xacro:property name="laser_scanner_height" value="0.1" />
-    <xacro:property name="laser_scanner_length" value="0.1" />
     <link name="laser_scanner">
         <inertial>
@@ -11,7 +8,7 @@
         </inertial>
         <visual>
-            <origin xyz="0 0 0" rpy="0 0 0"/>
-            <geometry>
-                <box size="${laser_scanner_width} ${laser_scanner_length} ${laser_scanner_height}" />
+            <origin xyz="0 0 0" rpy="${pi} 0 0"/>
+            <geometry name="lms100">
+                <mesh filename="package://tbd_podi_description/meshes/sick-lms1xx.dae"/>
             </geometry>
             <material name="laser_scanner_color">
@@ -20,7 +17,7 @@
         </visual>
         <collision>
-            <origin xyz="0 0 0" rpy="0 0 0"/>
-            <geometry>
-                <box size="${laser_scanner_width} ${laser_scanner_length} ${laser_scanner_height}" />
+            <origin xyz="0 0 0" rpy="${pi} 0 0"/>
+            <geometry name="lms100">
+                <mesh filename="package://tbd_podi_description/meshes/sick-lms1xx.dae"/>
             </geometry>
         </collision>
@@ -91,7 +88,4 @@
         <child link="podi_display"/>
     </joint>
-    <xacro:property name="camera_width" value="0.05" />
-    <xacro:property name="camera_height" value="0.05" />
-    <xacro:property name="camera_length" value="0.05" />
     <link name="podi_front_camera">
         <inertial>
@@ -102,6 +96,6 @@
         <visual>
             <origin xyz="0 0 0" rpy="0 0 0"/>
-            <geometry>
-                <box size="${camera_length} ${camera_width} ${camera_height}" />
+            <geometry name="zed">
+                <mesh filename="package://tbd_podi_description/meshes/zed.stl"/>
             </geometry>
             <material name="laser_scanner_color">
@@ -111,11 +105,11 @@
         <collision>
             <origin xyz="0 0 0" rpy="0 0 0"/>
-            <geometry>
-                <box size="${camera_length} ${camera_width} ${camera_height}" />
+            <geometry name="zed">
+                <mesh filename="package://tbd_podi_description/meshes/zed.stl"/>
             </geometry>
         </collision>
     </link>
    <joint name="camera_to_screen_joint" type="fixed">
-        <origin xyz="0 0 ${podi_face_screen_height + 0.01}" rpy="0 0 0"/>
+        <origin xyz="0 0 ${podi_face_screen_height/2 + 0.025}" rpy="0 0 0"/>
         <axis xyz="0 1 0"/>
         <parent link="podi_face_screen"/>
