Commit message: Added tbd_podi_face component

File: tbd_podi_description/urdf/podi.gazebo.xacro (robot description, xacro)
@@ -37,5 +37,5 @@
         <height>1080</height>
         <width>1920</width>
-        <topicName>/podi_screen</topicName>
+        <topicName>/podi/screen_face</topicName>
       </plugin>
     </visual>

File: tbd_podi_description/urdf/podi.urdf (robot description, URDF)
Before this commit: robot podi, 20 links, 19 joints
Joints:
- joint camera_to_screen_joint: origin xyz=0 0 0.21 rpy=0 0 0 -> xyz=0 0 0.21000000000000002 rpy=0 0 0

Commit message: fixed laser's incorrect frame and topic

File: tbd_podi_description/urdf/podi.gazebo.xacro (robot description, xacro)
@@ -13,8 +13,8 @@
       <publishWheelTF>false</publishWheelTF>
       <wheelAcceleration>1.8</wheelAcceleration>
-      <commandTopic>cmd_vel</commandTopic>
+      <commandTopic>${robotname}/cmd_vel</commandTopic>
       <robotBaseFrame>base_link</robotBaseFrame>
-      <odometryTopic>odom</odometryTopic>
-      <odometryFrame>odom</odometryFrame>
+      <odometryTopic>${robotname}/odom</odometryTopic>
+      <odometryFrame>${robotname}_odom</odometryFrame>
       <odometrySource>encoder</odometrySource>      <!-- The options are world and encoder. World means getting it straight from Gazebo -->
     </plugin>
@@ -24,5 +24,5 @@
       <updateRate>100.0</updateRate>
       <bodyName>base_link</bodyName>
-      <topicName>pose_ground_truth</topicName>
+      <topicName>${robotname}/pose_ground_truth</topicName>
       <gaussianNoise>0.01</gaussianNoise>
       <frameName>map</frameName>
@@ -31,5 +31,5 @@
     </plugin>
   </gazebo>
-  <gazebo reference="laser_scanner">
+  <gazebo reference="${robotname}_laser_scanner">
     <sensor type="gpu_ray" name="lms100x">
       <pose>0 0 0 0 0 0</pose>
@@ -57,19 +57,19 @@
       </ray>
       <plugin name="gazebo_ros_head_hokuyo_controller" filename="libgazebo_ros_gpu_laser.so">
-        <topicName>/scan</topicName>
-        <frameName>laser_scanner</frameName>
+        <topicName>${robotname}/scan</topicName>
+        <frameName>${robotname}_laser_scanner</frameName>
       </plugin>
     </sensor>
   </gazebo>
-  <gazebo reference="podi_display">
+  <gazebo reference="${robotname}_display">
     <visual>
       <plugin name="screen_video_controller" filename="libgazebo_ros_video.so">
         <height>1080</height>
         <width>1920</width>
-        <topicName>/podi/screen_face</topicName>
+        <topicName>${robotname}/screen_face</topicName>
       </plugin>
     </visual>
   </gazebo>
-  <gazebo reference="podi_front_camera">
+  <gazebo reference="${robotname}_front_camera">
     <sensor type="camera" name="front_camera">
       <update_rate>30.0</update_rate>
@@ -97,8 +97,8 @@
         <alwaysOn>true</alwaysOn>
         <updateRate>0.0</updateRate>
-        <cameraName>/front_camera</cameraName>
-        <imageTopicName>image_raw</imageTopicName>
+        <cameraName>front_camera</cameraName>
+        <imageTopicName>${robotname}/image_raw</imageTopicName>
         <cameraInfoTopicName>camera_info</cameraInfoTopicName>
-        <frameName>podi_front_camera</frameName>
+        <frameName>${robotname}_front_camera</frameName>
         <hackBaseline>0.07</hackBaseline>
         <distortionK1>0.0</distortionK1>

File: tbd_podi_description/urdf/podi.urdf.xacro (robot description, xacro)
@@ -2,4 +2,5 @@
 <robot name="podi"
     xmlns:xacro="http://ros.org/wiki/xacro">
+    <xacro:property name="robotname" value="podi" />
     <!-- Inport inertia functions -->
     <xacro:include filename="$(find tbd_podi_description)/urdf/inertia_tensors.xacro"/>

File: tbd_podi_description/urdf/podi_handle.xacro (robot description, xacro)
@@ -2,9 +2,5 @@
 <robot xmlns:xacro="http://ros.org/wiki/xacro">
     <link name="handle_base">
-        <inertial>
-            <mass value="1" />
-            <origin xyz="0 0 0" />
-            <inertia ixx="1" ixy="0" ixz="0" iyy="1" iyz="0" izz="1" />
-        </inertial>
+        <xacro:cylinder_inertial radius="0.06" length="0.04" mass="10" />
         <visual>
             <origin xyz="0 0 0.02" rpy="0 0 0"/>

File: tbd_podi_description/urdf/podi_structure.xacro (robot description, xacro)
@@ -1,5 +1,5 @@
 <?xml version="1.0"?>
 <robot xmlns:xacro="http://ros.org/wiki/xacro">
-    <link name="laser_scanner">
+    <link name="${robotname}_laser_scanner">
         <inertial>
             <mass value="1" />
@@ -8,5 +8,5 @@
         </inertial>
         <visual>
-            <origin xyz="0 0 0" rpy="${pi} 0 0"/>
+            <origin xyz="0 0 0" rpy="0 0 0"/>
             <geometry name="lms100">
                 <mesh filename="package://tbd_podi_description/meshes/sick-lms1xx.dae"/>
@@ -17,5 +17,5 @@
         </visual>
         <collision>
-            <origin xyz="0 0 0" rpy="${pi} 0 0"/>
+            <origin xyz="0 0 0" rpy="0 0 0"/>
             <geometry name="lms100">
                 <mesh filename="package://tbd_podi_description/meshes/sick-lms1xx.dae"/>
@@ -23,13 +23,13 @@
         </collision>
     </link>
-    <joint name="laser_scanner_to_base_joint" type="fixed">
-        <origin xyz="0.015 0 0.15" rpy="0 0 0"/>
+    <joint name="${robotname}_laser_scanner_to_base_joint" type="fixed">
+        <origin xyz="0.015 0 0.15" rpy="${pi} 0 0"/>
         <parent link="back_sonar"/>
-        <child link="laser_scanner"/>
+        <child link="${robotname}_laser_scanner"/>
     </joint>
-    <xacro:property name="podi_face_screen_width" value="0.01" />
-    <xacro:property name="podi_face_screen_height" value="0.2" />
-    <xacro:property name="podi_face_screen_length" value="0.2" />
-    <link name="podi_face_screen">
+    <xacro:property name="face_screen_width" value="0.01" />
+    <xacro:property name="face_screen_height" value="0.2" />
+    <xacro:property name="face_screen_length" value="0.2" />
+    <link name="${robotname}_face_screen">
         <inertial>
             <mass value="0.5" />
@@ -40,7 +40,7 @@
             <origin xyz="0 0 0" rpy="0 0 0"/>
             <geometry>
-                <box size="${podi_face_screen_width} ${podi_face_screen_length} ${podi_face_screen_height}" />
+                <box size="${face_screen_width} ${face_screen_length} ${face_screen_height}" />
             </geometry>
-            <material name="laser_scanner_color">
+            <material name="face_screen_color">
                 <color rgba="1 1 1 1"/>
             </material>
@@ -49,17 +49,17 @@
             <origin xyz="0 0 0" rpy="0 0 0"/>
             <geometry>
-                <box size="${podi_face_screen_width} ${podi_face_screen_length} ${podi_face_screen_height}" />
+                <box size="${face_screen_width} ${face_screen_length} ${face_screen_height}" />
             </geometry>
         </collision>
     </link>
     <joint name="screen_to_laser_scanner_joint" type="fixed">
-        <origin xyz="0.0 0 ${podi_face_screen_height + 0.05}" rpy="0 0 0"/>
-        <parent link="laser_scanner"/>
-        <child link="podi_face_screen"/>
+        <origin xyz="0.0 0 ${0.15 + face_screen_height + 0.05}" rpy="0 0 0"/>
+        <parent link="back_sonar"/>
+        <child link="${robotname}_face_screen"/>
     </joint>
-    <xacro:property name="podi_display_width" value="0.01" />
-    <xacro:property name="podi_display_height" value="0.10125" />
-    <xacro:property name="podi_display_length" value="0.18" />
-    <link name="podi_display">
+    <xacro:property name="display_width" value="0.01" />
+    <xacro:property name="display_height" value="0.10125" />
+    <xacro:property name="display_length" value="0.18" />
+    <link name="${robotname}_display">
         <inertial>
             <mass value="0.01" />
@@ -70,7 +70,7 @@
             <origin xyz="0 0 0" rpy="0 0 0"/>
             <geometry>
-                <box size=" ${podi_display_length} ${podi_display_height} ${podi_display_width}" />
+                <box size=" ${display_length} ${display_height} ${display_width}" />
             </geometry>
-            <material name="podi_display_color">
+            <material name="${robotname}_display_color">
                 <color rgba="0 0 0 1"/>
             </material>
@@ -79,5 +79,5 @@
             <origin xyz="0 0 0" rpy="0 0 0"/>
             <geometry>
-                <box size=" ${podi_display_length} ${podi_display_height} ${podi_display_width}" />
+                <box size=" ${display_length} ${display_height} ${display_width}" />
             </geometry>
         </collision>
@@ -85,8 +85,8 @@
     <joint name="display_to_screen_joint" type="fixed">
         <origin xyz="0.01 0 0" rpy="${3.1415927/2.0} 0 ${3.1415927/2.0}"/>
-        <parent link="podi_face_screen"/>
-        <child link="podi_display"/>
+        <parent link="${robotname}_face_screen"/>
+        <child link="${robotname}_display"/>
     </joint>
-    <link name="podi_front_camera">
+    <link name="${robotname}_front_camera">
         <inertial>
             <mass value="0.01" />
@@ -111,8 +111,8 @@
     </link>
    <joint name="camera_to_screen_joint" type="fixed">
-        <origin xyz="0 0 ${podi_face_screen_height/2 + 0.025}" rpy="0 0 0"/>
+        <origin xyz="0 0 ${face_screen_height/2 + 0.025}" rpy="0 0 0"/>
         <axis xyz="0 1 0"/>
-        <parent link="podi_face_screen"/>
-        <child link="podi_front_camera"/>
+        <parent link="${robotname}_face_screen"/>
+        <child link="${robotname}_front_camera"/>
     </joint>
 </robot>

Commit message: Fixed laser & change topic name

File: tbd_podi_description/urdf/podi.gazebo.xacro (robot description, xacro)
@@ -31,21 +31,21 @@
     </plugin>
   </gazebo>
-  <gazebo reference="${robotname}_laser_scanner">
+  <gazebo reference="laser_scanner">
     <sensor type="gpu_ray" name="lms100x">
       <pose>0 0 0 0 0 0</pose>
       <!-- <visualize>false</visualize> -->
-      <update_rate>20</update_rate>
+      <update_rate>25</update_rate>
       <ray>
         <scan>
           <horizontal>
-            <samples>360</samples>
-            <resolution>1</resolution>
-            <min_angle>-1.570796</min_angle>
-            <max_angle>1.570796</max_angle>
+            <samples>540</samples>
+            <resolution>0.5</resolution>
+            <min_angle>-2.35619</min_angle>
+            <max_angle>2.35619</max_angle>
           </horizontal>
         </scan>
         <range>
-          <min>0.10</min>
-          <max>30.0</max>
+          <min>0.5</min>
+          <max>20.0</max>
           <resolution>0.01</resolution>
         </range>
@@ -57,6 +57,7 @@
       </ray>
       <plugin name="gazebo_ros_head_hokuyo_controller" filename="libgazebo_ros_gpu_laser.so">
-        <topicName>${robotname}/scan</topicName>
-        <frameName>${robotname}_laser_scanner</frameName>
+        <topicName>laser</topicName>
+        <frameName>laser_scanner</frameName>
+        <robotNamespace>${robotname}</robotNamespace>
       </plugin>
     </sensor>

File: tbd_podi_description/urdf/podi_structure.xacro (robot description, xacro)
@@ -1,5 +1,5 @@
 <?xml version="1.0"?>
 <robot xmlns:xacro="http://ros.org/wiki/xacro">
-    <link name="${robotname}_laser_scanner">
+    <link name="laser_scanner">
         <inertial>
             <mass value="1" />
@@ -23,8 +23,8 @@
         </collision>
     </link>
-    <joint name="${robotname}_laser_scanner_to_base_joint" type="fixed">
+    <joint name="laser_scanner_to_base_joint" type="fixed">
         <origin xyz="0.015 0 0.15" rpy="${pi} 0 0"/>
         <parent link="back_sonar"/>
-        <child link="${robotname}_laser_scanner"/>
+        <child link="laser_scanner"/>
     </joint>
     <xacro:property name="face_screen_width" value="0.01" />

Commit message: 1.1.5 -  Podi Inertia Model Teakers. (#12)
* tweaked inertia

* Added Azure Kinect

File: tbd_podi_description/urdf/podi.gazebo.xacro (robot description, xacro)
@@ -12,5 +12,5 @@
       <publishWheelJointState>true</publishWheelJointState>
       <publishWheelTF>false</publishWheelTF>
-      <wheelAcceleration>1.8</wheelAcceleration>
+      <wheelAcceleration>1</wheelAcceleration>
       <commandTopic>cmd_vel</commandTopic>
       <odometryTopic>odom</odometryTopic>
@@ -67,6 +67,6 @@
     <visual>
       <plugin name="screen_video_controller" filename="libgazebo_ros_video.so">
-        <height>1080</height>
-        <width>1920</width>
+        <height>1280</height>
+        <width>720</width>
         <topicName>screen_face</topicName>
         <robotNamespace>${robotname}</robotNamespace>
@@ -74,38 +74,20 @@
     </visual>
   </gazebo>
-  <gazebo reference="${robotname}_front_camera">
-    <sensor type="camera" name="front_camera">
+  <gazebo reference="camera_base">
+    <sensor type="depth" name="front_depth_camera">
       <update_rate>30.0</update_rate>
-      <camera name="head">
+      <camera name="front_camera">
         <horizontal_fov>1.57079632679</horizontal_fov>
         <image>
-          <width>2560</width>
-          <height>720</height>
+          <width>1920</width>
+          <height>1080</height>
           <format>R8G8B8</format>
         </image>
-        <clip>
-          <near>0.02</near>
-          <far>300</far>
-        </clip>
-        <noise>
-          <type>gaussian</type>
-          <mean>0.0</mean>
-          <stddev>0.007</stddev>
-        </noise>
       </camera>
-      <plugin name="camera_controller" filename="libgazebo_ros_camera.so">
-        <alwaysOn>true</alwaysOn>
-        <updateRate>0.0</updateRate>
-        <cameraName>front_camera</cameraName>
-        <imageTopicName>image_raw</imageTopicName>
-        <cameraInfoTopicName>camera_info</cameraInfoTopicName>
-        <frameName>${robotname}_front_camera</frameName>
+      <plugin name="head_depth_camera" filename="libgazebo_ros_depth_camera.so">
+        <cameraName>azure_kinect</cameraName>
+        <frameName>camera_point</frameName>
         <robotNamespace>${robotname}</robotNamespace>
-        <hackBaseline>0.07</hackBaseline>
-        <distortionK1>0.0</distortionK1>
-        <distortionK2>0.0</distortionK2>
-        <distortionK3>0.0</distortionK3>
-        <distortionT1>0.0</distortionT1>
-        <distortionT2>0.0</distortionT2>
+        <pointCloudCutoff>2.0</pointCloudCutoff>
       </plugin>
     </sensor>

File: tbd_podi_description/urdf/podi_structure.xacro (robot description, xacro)
@@ -2,9 +2,5 @@
 <robot xmlns:xacro="http://ros.org/wiki/xacro">
     <link name="laser_scanner">
-        <inertial>
-            <mass value="1" />
-            <origin xyz="0 0 0" />
-            <inertia ixx="1" ixy="0" ixz="0" iyy="1" iyz="0" izz="1" />
-        </inertial>
+        <xacro:box_inertial x="0.105" y="0.102" z="0.152" mass="0.429" />
         <visual>
             <origin xyz="0 0 0" rpy="0 0 0"/>
@@ -28,13 +24,9 @@
         <child link="laser_scanner"/>
     </joint>
-    <xacro:property name="face_screen_width" value="0.01" />
-    <xacro:property name="face_screen_height" value="0.2" />
-    <xacro:property name="face_screen_length" value="0.2" />
+    <xacro:property name="face_screen_width" value="0.006" />
+    <xacro:property name="face_screen_height" value="0.2373" />
+    <xacro:property name="face_screen_length" value="0.169" />
     <link name="${robotname}_face_screen">
-        <inertial>
-            <mass value="0.5" />
-            <origin xyz="0 0 0" />
-            <inertia ixx="1" ixy="0" ixz="0" iyy="1" iyz="0" izz="1" />
-        </inertial>
+        <xacro:box_inertial x="${face_screen_width}" y="${face_screen_length}" z="${face_screen_height}" mass="0.429" />
         <visual>
             <origin xyz="0 0 0" rpy="0 0 0"/>
@@ -100,31 +92,18 @@
         <child link="${robotname}_display"/>
     </joint>
-    <link name="${robotname}_front_camera">
+    <link name="${robotname}_camera_mount">
         <inertial>
-            <mass value="0.01" />
+            <mass value="0.0001" />
             <origin xyz="0 0 0" />
             <inertia ixx="1" ixy="0" ixz="0" iyy="1" iyz="0" izz="1" />
         </inertial>
-        <visual>
-            <origin xyz="0 0 0" rpy="0 0 0"/>
-            <geometry name="zed">
-                <mesh filename="package://tbd_podi_description/meshes/zed.stl"/>
-            </geometry>
-            <material name="laser_scanner_color">
-                <color rgba="1 1 1 1"/>
-            </material>
-        </visual>
-        <collision>
-            <origin xyz="0 0 0" rpy="0 0 0"/>
-            <geometry name="zed">
-                <mesh filename="package://tbd_podi_description/meshes/zed.stl"/>
-            </geometry>
-        </collision>
     </link>
-   <joint name="camera_to_screen_joint" type="fixed">
-        <origin xyz="0 0 ${face_screen_height/2 + 0.025}" rpy="0 0 0"/>
+   <joint name="camera_mount_to_screen_joint" type="fixed">
+        <origin xyz="0.025 0 ${face_screen_height/2 + 0.025}" rpy="0 0 0"/>
         <axis xyz="0 1 0"/>
         <parent link="${robotname}_face_screen"/>
-        <child link="${robotname}_front_camera"/>
+        <child link="${robotname}_camera_mount"/>
     </joint>
+    <!-- Include Azure Kinect -->
+    <xacro:insert_azure_kinect parent="${robotname}_camera_mount" tf_prefix=""/>
 </robot>
