Commit message: made podi struct more accurate

File: tbd_podi_description/urdf/podi_structure.xacro (robot description, xacro)
@@ -25,6 +25,6 @@
     </joint>
     <xacro:property name="face_screen_width" value="0.006" />
-    <xacro:property name="face_screen_height" value="0.2373" />
-    <xacro:property name="face_screen_length" value="0.169" />
+    <xacro:property name="face_screen_height" value="0.169" />
+    <xacro:property name="face_screen_length" value="0.2373" />
     <link name="$(arg robot_name)_face_screen">
         <xacro:box_inertial x="${face_screen_width}" y="${face_screen_length}" z="${face_screen_height}" mass="0.429" />
@@ -58,11 +58,11 @@
     </joint>
     <joint name="screen_to_$(arg robot_name)_laser_scanner_joint" type="fixed">
-        <origin xyz="0.0 0 ${0.15 + face_screen_height + 0.05}" rpy="0 0 0"/>
+        <origin xyz="0.0 0.0 ${0.025 + 0.4953}" rpy="0 0 0"/>
         <parent link="$(arg robot_name)_back_sonar"/>
         <child link="$(arg robot_name)_head"/>
     </joint>
     <xacro:property name="display_width" value="0.01" />
-    <xacro:property name="display_height" value="0.10125" />
-    <xacro:property name="display_length" value="0.18" />
+    <xacro:property name="display_height" value="0.147" />
+    <xacro:property name="display_length" value="0.197" />
     <link name="$(arg robot_name)_display">
         <inertial>
@@ -93,7 +93,7 @@
     </joint>
    <joint name="$(arg robot_name)_camera_mount_to_screen_joint" type="fixed">
-        <origin xyz="0.025 0 ${face_screen_height/2 + 0.025}" rpy="0 0 0"/>
+        <origin xyz="0.0 0.0 0.1016" rpy="0 0 0"/>
         <axis xyz="0 1 0"/>
-        <parent link="$(arg robot_name)_face_screen"/>
+        <parent link="$(arg robot_name)_head"/>
         <child link="$(arg robot_name)_front_camera_mount"/>
     </joint>

Commit message: update podi structure

File: tbd_podi_description/urdf/podi_structure.xacro (robot description, xacro)
@@ -1,4 +1,12 @@
 <?xml version="1.0"?>
 <robot xmlns:xacro="http://ros.org/wiki/xacro">
+    <!-- The size of the tablet -->
+    <xacro:property name="face_screen_width" value="0.006" />
+    <xacro:property name="face_screen_height" value="0.169" />
+    <xacro:property name="face_screen_length" value="0.2373" />
+    <!-- The size of the screen on th etable -->
+    <xacro:property name="display_width" value="0.01" />
+    <xacro:property name="display_height" value="0.147" />
+    <xacro:property name="display_length" value="0.197" />
     <link name="$(arg robot_name)_laser_scanner">
         <xacro:box_inertial x="0.105" y="0.102" z="0.152" mass="0.429" />
@@ -24,7 +32,45 @@
         <child link="$(arg robot_name)_laser_scanner"/>
     </joint>
-    <xacro:property name="face_screen_width" value="0.006" />
-    <xacro:property name="face_screen_height" value="0.169" />
-    <xacro:property name="face_screen_length" value="0.2373" />
+    <link name="$(arg robot_name)_head_bottom_bar">
+        <xacro:box_inertial x="0.0254" y="0.3048" z="0.0254" mass="0.1" />
+        <visual>
+            <origin xyz="0 0 0" rpy="0 0 0"/>
+            <geometry>
+                <box size=" 0.0254 0.3048 0.0254" />
+            </geometry>
+            <material name="$display_color">
+                <color rgba="1 1 1 1"/>
+            </material>
+        </visual>
+    </link>
+    <joint name="$(arg robot_name)_head_bottom_bar_to_base_joint" type="fixed">
+        <origin xyz="0.1651 0 ${0.234 + 0.3175}" rpy="0 0 0"/>
+        <parent link="$(arg robot_name)_base_link"/>
+        <child link="$(arg robot_name)_head_bottom_bar"/>
+    </joint>
+    <link name="$(arg robot_name)_head_mount">
+        <inertial>
+            <mass value="0.01" />
+            <origin xyz="0 0 0" />
+            <inertia ixx="1" ixy="0" ixz="0" iyy="1" iyz="0" izz="1" />
+        </inertial>
+    </link>
+    <joint name="$(arg robot_name)_head_mount_to_head_bottom_bar" type="fixed">
+        <origin xyz="${0.0254} 0.0 ${0.0889}" rpy="0 0 0"/>
+        <parent link="$(arg robot_name)_head_bottom_bar"/>
+        <child link="$(arg robot_name)_head_mount"/>
+    </joint>
+    <link name="$(arg robot_name)_head">
+        <inertial>
+            <mass value="0.01" />
+            <origin xyz="0 0 0" />
+            <inertia ixx="1" ixy="0" ixz="0" iyy="1" iyz="0" izz="1" />
+        </inertial>
+    </link>
+    <joint name="$(arg robot_name)_head_to_head_mount" type="fixed">
+        <origin xyz="0 0 ${face_screen_height/2}" rpy="0 0 0"/>
+        <parent link="$(arg robot_name)_head_mount"/>
+        <child link="$(arg robot_name)_head"/>
+    </joint>
     <link name="$(arg robot_name)_face_screen">
         <xacro:box_inertial x="${face_screen_width}" y="${face_screen_length}" z="${face_screen_height}" mass="0.429" />
@@ -45,11 +91,4 @@
         </collision>
     </link>
-    <link name="$(arg robot_name)_head">
-        <inertial>
-            <mass value="0.01" />
-            <origin xyz="0 0 0" />
-            <inertia ixx="1" ixy="0" ixz="0" iyy="1" iyz="0" izz="1" />
-        </inertial>
-    </link>
     <joint name="$(arg robot_name)_head_to_screen_joint" type="fixed">
         <origin xyz="0 0 0" rpy="0 0 0"/>
@@ -57,12 +96,4 @@
         <child link="$(arg robot_name)_face_screen"/>
     </joint>
-    <joint name="screen_to_$(arg robot_name)_laser_scanner_joint" type="fixed">
-        <origin xyz="0.0 0.0 ${0.025 + 0.4953}" rpy="0 0 0"/>
-        <parent link="$(arg robot_name)_back_sonar"/>
-        <child link="$(arg robot_name)_head"/>
-    </joint>
-    <xacro:property name="display_width" value="0.01" />
-    <xacro:property name="display_height" value="0.147" />
-    <xacro:property name="display_length" value="0.197" />
     <link name="$(arg robot_name)_display">
         <inertial>
@@ -92,11 +123,29 @@
         <child link="$(arg robot_name)_display"/>
     </joint>
-   <joint name="$(arg robot_name)_camera_mount_to_screen_joint" type="fixed">
-        <origin xyz="0.0 0.0 0.1016" rpy="0 0 0"/>
-        <axis xyz="0 1 0"/>
-        <parent link="$(arg robot_name)_head"/>
-        <child link="$(arg robot_name)_front_camera_mount"/>
+    <link name="$(arg robot_name)_head_top_bar">
+        <xacro:box_inertial x="0.0254" y="0.3048" z="0.0254" mass="0.1" />
+        <visual>
+            <origin xyz="0 0 0" rpy="0 0 0"/>
+            <geometry>
+                <box size=" 0.0254 0.3048 0.0254" />
+            </geometry>
+            <material name="$display_color">
+                <color rgba="1 1 1 1"/>
+            </material>
+        </visual>
+    </link>
+    <joint name="$(arg robot_name)_head_top_bar_to_head_bottom_bar" type="fixed">
+        <origin xyz="0 0 ${0.254}" rpy="0 0 0"/>
+        <parent link="$(arg robot_name)_head_bottom_bar"/>
+        <child link="$(arg robot_name)_head_top_bar"/>
     </joint>
-    <xacro:arg name="base_frame" default="$(arg robot_name)_front_camera_mount"/>
+    <!-- Note that the baseframe is created by the ZED URDF -->
+   <joint name="$(arg robot_name)_head_camera_mount_to_head_top_bar" type="fixed">
+        <origin xyz="0 0 ${0.0127 + 0.03/2}" rpy="0 0 0"/>
+        <axis xyz="0 0 0"/>
+        <parent link="$(arg robot_name)_head_top_bar"/>
+        <child link="$(arg robot_name)_head_camera_mount"/>
+    </joint>
+    <xacro:arg name="base_frame" default="$(arg robot_name)_head_camera_mount"/>
     <xacro:arg name="camera_model" default="zed2"/>
     <xacro:arg name="camera_name" default="$(arg robot_name)_front_camera"/>

Commit message: added marker

File: tbd_podi_description/urdf/podi_structure.xacro (robot description, xacro)
@@ -31,4 +31,21 @@
         <parent link="$(arg robot_name)_back_sonar"/>
         <child link="$(arg robot_name)_laser_scanner"/>
+    </joint>
+    <link name="$(arg robot_name)_calibration_marker">
+        <xacro:box_inertial x="0.1524" y="0.1524" z="0.01" mass="0.1" />
+        <visual>
+            <origin xyz="${0.1524/2} ${0.1524/2} 0" rpy="0 0 0"/>
+            <geometry>
+                <box size=" 0.1524 0.1524 0.1" />
+            </geometry>
+            <material name="$display_color">
+                <color rgba="1 1 1 1"/>
+            </material>
+        </visual>
+    </link>
+    <joint name="$(arg robot_name)_calibration_marker_to_base_joint" type="fixed">
+        <origin xyz="0 0.1524 ${0.234 + 0.1524}" rpy="0 0 0"/>
+        <parent link="$(arg robot_name)_base_link"/>
+        <child link="$(arg robot_name)_head_bottom_bar"/>
     </joint>
     <link name="$(arg robot_name)_head_bottom_bar">

Commit message: fix calibration_marker

File: tbd_podi_description/urdf/podi_structure.xacro (robot description, xacro)
@@ -37,5 +37,5 @@
             <origin xyz="${0.1524/2} ${0.1524/2} 0" rpy="0 0 0"/>
             <geometry>
-                <box size=" 0.1524 0.1524 0.1" />
+                <box size=" 0.1524 0.1524 0.01" />
             </geometry>
             <material name="$display_color">
@@ -45,7 +45,7 @@
     </link>
     <joint name="$(arg robot_name)_calibration_marker_to_base_joint" type="fixed">
-        <origin xyz="0 0.1524 ${0.234 + 0.1524}" rpy="0 0 0"/>
+        <origin xyz="0 0.1524 ${0.234 + 0.1524}" rpy="-${pi/2} ${pi/2} 0 "/>
         <parent link="$(arg robot_name)_base_link"/>
-        <child link="$(arg robot_name)_head_bottom_bar"/>
+        <child link="$(arg robot_name)_calibration_marker"/>
     </joint>
     <link name="$(arg robot_name)_head_bottom_bar">

Commit message: fix urdf

File: tbd_podi_description/urdf/podi_structure.xacro (robot description, xacro)
@@ -45,5 +45,5 @@
     </link>
     <joint name="$(arg robot_name)_calibration_marker_to_base_joint" type="fixed">
-        <origin xyz="0 0.1524 ${0.234 + 0.1524}" rpy="-${pi/2} ${pi/2} 0 "/>
+        <origin xyz="0 0.1524 ${0.234 + 0.3048}" rpy="-${pi/2} ${pi/2} 0 "/>
         <parent link="$(arg robot_name)_base_link"/>
         <child link="$(arg robot_name)_calibration_marker"/>

Commit message: new map!

File: tbd_podi_description/urdf/podi_structure.xacro (robot description, xacro)
@@ -45,5 +45,5 @@
     </link>
     <joint name="$(arg robot_name)_calibration_marker_to_base_joint" type="fixed">
-        <origin xyz="0 0.1524 ${0.234 + 0.3048}" rpy="-${pi/2} ${pi/2} 0 "/>
+        <origin xyz="0 ${0.1524 + 0.003} ${0.234 + 0.3175}" rpy="-${pi/2} ${pi/2} 0 "/>
         <parent link="$(arg robot_name)_base_link"/>
         <child link="$(arg robot_name)_calibration_marker"/>

Commit message: map + URDF update

File: tbd_podi_description/urdf/podi_structure.xacro (robot description, xacro)
@@ -28,14 +28,14 @@
     </link>
     <joint name="$(arg robot_name)_laser_scanner_to_base_joint" type="fixed">
-        <origin xyz="0.015 0 0.15" rpy="${pi} 0 0"/>
-        <parent link="$(arg robot_name)_back_sonar"/>
+        <origin xyz="${0.046 + 0.0545} 0 ${0.234 + 0.1524 - 0.008 - 0.0367}" rpy="${pi} 0 0"/>
+        <parent link="$(arg robot_name)_base_link"/>
         <child link="$(arg robot_name)_laser_scanner"/>
     </joint>
     <link name="$(arg robot_name)_calibration_marker">
-        <xacro:box_inertial x="0.1524" y="0.1524" z="0.01" mass="0.1" />
+        <xacro:box_inertial x="0.1651" y="0.2921" z="0.01" mass="0.1" />
         <visual>
-            <origin xyz="${0.1524/2} ${0.1524/2} 0" rpy="0 0 0"/>
+            <origin xyz="${0.1651/2} ${0.2921/2} 0" rpy="0 0 0"/>
             <geometry>
-                <box size=" 0.1524 0.1524 0.01" />
+                <box size="0.1651 0.2921 0.01" />
             </geometry>
             <material name="$display_color">
@@ -45,5 +45,5 @@
     </link>
     <joint name="$(arg robot_name)_calibration_marker_to_base_joint" type="fixed">
-        <origin xyz="0 ${0.1524 + 0.003} ${0.234 + 0.3175}" rpy="-${pi/2} ${pi/2} 0 "/>
+        <origin xyz="${-0.1651 + 0.02} ${0.1463 + 0.007} ${0.234 + 0.3048 + 0.008}" rpy="-${pi/2} -${pi/2} 0 "/>
         <parent link="$(arg robot_name)_base_link"/>
         <child link="$(arg robot_name)_calibration_marker"/>

Commit message: changing URDF

File: tbd_podi_description/urdf/podi_structure.xacro (robot description, xacro)
@@ -45,5 +45,5 @@
     </link>
     <joint name="$(arg robot_name)_calibration_marker_to_base_joint" type="fixed">
-        <origin xyz="${-0.1651 + 0.02} ${0.1463 + 0.007} ${0.234 + 0.3048 + 0.008}" rpy="-${pi/2} -${pi/2} 0 "/>
+        <origin xyz="${-0.1651 + 0.003 + 0.0061} ${-0.1463 - 0.007} ${0.234 + 0.3048 + 0.003 + 0.021}" rpy="-${pi/2} 0 0 "/>
         <parent link="$(arg robot_name)_base_link"/>
         <child link="$(arg robot_name)_calibration_marker"/>

Commit message: fix URDF

File: tbd_podi_description/urdf/podi_structure.xacro (robot description, xacro)
@@ -33,9 +33,9 @@
     </joint>
     <link name="$(arg robot_name)_calibration_marker">
-        <xacro:box_inertial x="0.1651" y="0.2921" z="0.01" mass="0.1" />
+        <xacro:box_inertial x="0.2921" y="0.1651" z="0.01" mass="0.1" />
         <visual>
-            <origin xyz="${0.1651/2} ${0.2921/2} 0" rpy="0 0 0"/>
+            <origin xyz="${0.2921/2} ${0.1651/2} 0" rpy="0 0 0"/>
             <geometry>
-                <box size="0.1651 0.2921 0.01" />
+                <box size="0.2921 0.1651 0.01" />
             </geometry>
             <material name="$display_color">
@@ -45,5 +45,5 @@
     </link>
     <joint name="$(arg robot_name)_calibration_marker_to_base_joint" type="fixed">
-        <origin xyz="${-0.1651 + 0.003 + 0.0061} ${-0.1463 - 0.007} ${0.234 + 0.3048 + 0.003 + 0.021}" rpy="-${pi/2} 0 0 "/>
+        <origin xyz="${-0.1651 + 0.003 + 0.0061} ${-0.1463 - 0.007} ${0.234 + 0.3048 + 0.003 + 0.021}" rpy="${pi/2} 0 0 "/>
         <parent link="$(arg robot_name)_base_link"/>
         <child link="$(arg robot_name)_calibration_marker"/>

Commit message: podi-laptop-last-commit

File: tbd_podi_description/urdf/podi_structure.xacro (robot description, xacro)
@@ -45,5 +45,5 @@
     </link>
     <joint name="$(arg robot_name)_calibration_marker_to_base_joint" type="fixed">
-        <origin xyz="${-0.1651 + 0.003 + 0.0061} ${-0.1463 - 0.007} ${0.234 + 0.3048 + 0.003 + 0.021}" rpy="${pi/2} 0 0 "/>
+        <origin xyz="${-0.085} ${0.1463 + 0.007} ${0.234 + 0.213}" rpy="${pi/2} ${-pi/2} ${pi}"/>
         <parent link="$(arg robot_name)_base_link"/>
         <child link="$(arg robot_name)_calibration_marker"/>
